Commit message: ros2 workspace with launch file for moveit and fakecontroller

File: ros2_ws/src/piper_ros/src/piper_moveit/piper_no_gripper_moveit/config/piper.ros2_control.xacro (robot description, xacro)
@@ -1,54 +1,73 @@
 <?xml version="1.0"?>
 <robot xmlns:xacro="http://www.ros.org/wiki/xacro">
-    <xacro:macro name="piper_ros2_control" params="name initial_positions_file">
-        <xacro:property name="initial_positions" value="${load_yaml(initial_positions_file)['initial_positions']}"/>
-        <ros2_control name="${name}" type="system">
-            <hardware>
-                <!-- By default, set up controllers for simulation. This won't work on real hardware -->
-                <plugin>mock_components/GenericSystem</plugin>
-            </hardware>
-            <joint name="joint1">
-                <command_interface name="position"/>
-                <state_interface name="position">
-                  <param name="initial_value">${initial_positions['joint1']}</param>
-                </state_interface>
-                <state_interface name="velocity"/>
-            </joint>
-            <joint name="joint2">
-                <command_interface name="position"/>
-                <state_interface name="position">
-                  <param name="initial_value">${initial_positions['joint2']}</param>
-                </state_interface>
-                <state_interface name="velocity"/>
-            </joint>
-            <joint name="joint3">
-                <command_interface name="position"/>
-                <state_interface name="position">
-                  <param name="initial_value">${initial_positions['joint3']}</param>
-                </state_interface>
-                <state_interface name="velocity"/>
-            </joint>
-            <joint name="joint4">
-                <command_interface name="position"/>
-                <state_interface name="position">
-                  <param name="initial_value">${initial_positions['joint4']}</param>
-                </state_interface>
-                <state_interface name="velocity"/>
-            </joint>
-            <joint name="joint5">
-                <command_interface name="position"/>
-                <state_interface name="position">
-                  <param name="initial_value">${initial_positions['joint5']}</param>
-                </state_interface>
-                <state_interface name="velocity"/>
-            </joint>
-            <joint name="joint6">
-                <command_interface name="position"/>
-                <state_interface name="position">
-                  <param name="initial_value">${initial_positions['joint6']}</param>
-                </state_interface>
-                <state_interface name="velocity"/>
-            </joint>
-        </ros2_control>
-    </xacro:macro>
+  <!--
+    Makro für ros2_control am Piper.
+    Params:
+      - name: Name des ros2_control-Blocks
+      - initial_positions_file: YAML mit Startwerten
+      - fake_hardware: "true" -> GenericSystem (Simulation), "false" -> Platzhalter für echte HW
+  -->
+  <xacro:macro name="piper_ros2_control" params="name initial_positions_file fake_hardware:=true">
+    <!-- YAML laden -->
+    <xacro:property name="initial_positions"
+                    value="${load_yaml(initial_positions_file)['initial_positions']}" />
+    <ros2_control name="${name}" type="system">
+      <!-- Hardware abhängig vom Schalter -->
+      <xacro:if value="${fake_hardware}">
+        <!-- SIM / Fake -->
+        <hardware>
+          <plugin>mock_components/GenericSystem</plugin>
+        </hardware>
+      </xacro:if>
+      <xacro:unless value="${fake_hardware}">
+        <!-- ECHTE HW: hier später echten Treiber eintragen -->
+        <hardware>
+          <!-- TODO: richtigen Plugin-Namen für die reale Piper-HW einsetzen -->
+          <plugin>your_real_hardware_plugin/Driver</plugin>
+        </hardware>
+      </xacro:unless>
+      <joint name="joint1">
+        <command_interface name="position"/>
+        <state_interface name="position">
+          <param name="initial_value">${initial_positions['joint1']}</param>
+        </state_interface>
+        <state_interface name="velocity"/>
+      </joint>
+      <joint name="joint2">
+        <command_interface name="position"/>
+        <state_interface name="position">
+          <param name="initial_value">${initial_positions['joint2']}</param>
+        </state_interface>
+        <state_interface name="velocity"/>
+      </joint>
+      <joint name="joint3">
+        <command_interface name="position"/>
+        <state_interface name="position">
+          <param name="initial_value">${initial_positions['joint3']}</param>
+        </state_interface>
+        <state_interface name="velocity"/>
+      </joint>
+      <joint name="joint4">
+        <command_interface name="position"/>
+        <state_interface name="position">
+          <param name="initial_value">${initial_positions['joint4']}</param>
+        </state_interface>
+        <state_interface name="velocity"/>
+      </joint>
+      <joint name="joint5">
+        <command_interface name="position"/>
+        <state_interface name="position">
+          <param name="initial_value">${initial_positions['joint5']}</param>
+        </state_interface>
+        <state_interface name="velocity"/>
+      </joint>
+      <joint name="joint6">
+        <command_interface name="position"/>
+        <state_interface name="position">
+          <param name="initial_value">${initial_positions['joint6']}</param>
+        </state_interface>
+        <state_interface name="velocity"/>
+      </joint>
+    </ros2_control>
+  </xacro:macro>
 </robot>

File: ros2_ws/src/piper_ros/src/piper_moveit/piper_no_gripper_moveit/config/piper.urdf.xacro (robot description, xacro)
@@ -1,9 +1,17 @@
 <?xml version="1.0"?>
 <robot xmlns:xacro="http://www.ros.org/wiki/xacro" name="piper">
+    <!-- bestehendes arg -->
     <xacro:arg name="initial_positions_file" default="initial_positions.yaml" />
+    <!-- Schalter aus der Launch: true = Simulation, false = echte HW -->
+    <xacro:arg name="fake_hardware" default="true"/>
     <!-- Import piper urdf file -->
     <xacro:include filename="$(find piper_description)/urdf/piper_no_gripper_description.xacro" />
     <!-- Import control_xacro -->
     <xacro:include filename="piper.ros2_control.xacro" />
-    <xacro:piper_ros2_control name="FakeSystem" initial_positions_file="$(arg initial_positions_file)"/>
+    <!-- ros2_control-Makro mit dem neuen Schalter aufrufen -->
+    <xacro:piper_ros2_control
+        name="piper_hw"
+        initial_positions_file="$(arg initial_positions_file)"
+        fake_hardware="$(arg fake_hardware)"
+    />
 </robot>
