Commit message: starting piper with gripper

File: ros2_ws/src/piper_ros/src/piper_description/urdf/piper_description.urdf (robot description, URDF)
Before this commit: robot piper, 10 links, 9 joints
Joints:
- joint joint8: axis 0 0 -1 -> 0 0 1; mimic (none) -> joint=joint7 multiplier=-1 offset=0

File: ros2_ws/src/piper_ros/src/piper_moveit/piper_no_gripper_moveit/config/piper.ros2_control.xacro (robot description, xacro)
@@ -21,5 +21,4 @@
       </xacro:if>
       <xacro:unless value="${fake_hardware}">
-        <!-- ECHTE HW: hier später echten Treiber eintragen -->
         <hardware>
           <!-- TODO: richtigen Plugin-Namen für die reale Piper-HW einsetzen -->

File: ros2_ws/src/piper_ros/src/piper_moveit/piper_with_gripper_moveit/config/piper.ros2_control.xacro (robot description, xacro)
@@ -1,61 +1,68 @@
 <?xml version="1.0"?>
 <robot xmlns:xacro="http://www.ros.org/wiki/xacro">
-    <xacro:macro name="piper_ros2_control" params="name initial_positions_file">
-        <xacro:property name="initial_positions" value="${load_yaml(initial_positions_file)['initial_positions']}"/>
-        <ros2_control name="${name}" type="system">
-            <hardware>
-                <!-- By default, set up controllers for simulation. This won't work on real hardware -->
-                <plugin>mock_components/GenericSystem</plugin>
-            </hardware>
-            <joint name="joint1">
-                <command_interface name="position"/>
-                <state_interface name="position">
-                  <param name="initial_value">${initial_positions['joint1']}</param>
-                </state_interface>
-                <state_interface name="velocity"/>
-            </joint>
-            <joint name="joint2">
-                <command_interface name="position"/>
-                <state_interface name="position">
-                  <param name="initial_value">${initial_positions['joint2']}</param>
-                </state_interface>
-                <state_interface name="velocity"/>
-            </joint>
-            <joint name="joint3">
-                <command_interface name="position"/>
-                <state_interface name="position">
-                  <param name="initial_value">${initial_positions['joint3']}</param>
-                </state_interface>
-                <state_interface name="velocity"/>
-            </joint>
-            <joint name="joint4">
-                <command_interface name="position"/>
-                <state_interface name="position">
-                  <param name="initial_value">${initial_positions['joint4']}</param>
-                </state_interface>
-                <state_interface name="velocity"/>
-            </joint>
-            <joint name="joint5">
-                <command_interface name="position"/>
-                <state_interface name="position">
-                  <param name="initial_value">${initial_positions['joint5']}</param>
-                </state_interface>
-                <state_interface name="velocity"/>
-            </joint>
-            <joint name="joint6">
-                <command_interface name="position"/>
-                <state_interface name="position">
-                  <param name="initial_value">${initial_positions['joint6']}</param>
-                </state_interface>
-                <state_interface name="velocity"/>
-            </joint>
-            <joint name="joint7">
-                <command_interface name="position"/>
-                <state_interface name="position">
-                  <param name="initial_value">${initial_positions['joint7']}</param>
-                </state_interface>
-                <state_interface name="velocity"/>
-            </joint>
-        </ros2_control>
-    </xacro:macro>
+  <xacro:macro name="piper_ros2_control" params="name initial_positions_file fake_hardware:=true">
+    <xacro:property name="initial_positions"
+                    value="${load_yaml(initial_positions_file)['initial_positions']}" />
+    <ros2_control name="${name}" type="system">
+      <xacro:if value="${fake_hardware}">
+        <hardware>
+          <plugin>mock_components/GenericSystem</plugin>
+        </hardware>
+      </xacro:if>
+      <xacro:unless value="${fake_hardware}">
+        <hardware>
+          <plugin>your_real_hardware_plugin/Driver</plugin>
+        </hardware>
+      </xacro:unless>
+      <joint name="joint1">
+        <command_interface name="position"/>
+        <state_interface name="position">
+          <param name="initial_value">${initial_positions['joint1']}</param>
+        </state_interface>
+        <state_interface name="velocity"/>
+      </joint>
+      <joint name="joint2">
+        <command_interface name="position"/>
+        <state_interface name="position">
+          <param name="initial_value">${initial_positions['joint2']}</param>
+        </state_interface>
+        <state_interface name="velocity"/>
+      </joint>
+      <joint name="joint3">
+        <command_interface name="position"/>
+        <state_interface name="position">
+          <param name="initial_value">${initial_positions['joint3']}</param>
+        </state_interface>
+        <state_interface name="velocity"/>
+      </joint>
+      <joint name="joint4">
+        <command_interface name="position"/>
+        <state_interface name="position">
+          <param name="initial_value">${initial_positions['joint4']}</param>
+        </state_interface>
+        <state_interface name="velocity"/>
+      </joint>
+      <joint name="joint5">
+        <command_interface name="position"/>
+        <state_interface name="position">
+          <param name="initial_value">${initial_positions['joint5']}</param>
+        </state_interface>
+        <state_interface name="velocity"/>
+      </joint>
+      <joint name="joint6">
+        <command_interface name="position"/>
+        <state_interface name="position">
+          <param name="initial_value">${initial_positions['joint6']}</param>
+        </state_interface>
+        <state_interface name="velocity"/>
+      </joint>
+      <joint name="joint7">
+        <command_interface name="position"/>
+        <state_interface name="position">
+          <param name="initial_value">${initial_positions['joint7']}</param>
+        </state_interface>
+        <state_interface name="velocity"/>
+      </joint>
+    </ros2_control>
+  </xacro:macro>
 </robot>

File: ros2_ws/src/piper_ros/src/piper_moveit/piper_with_gripper_moveit/config/piper.urdf.xacro (robot description, xacro)
@@ -1,9 +1,15 @@
 <?xml version="1.0"?>
 <robot xmlns:xacro="http://www.ros.org/wiki/xacro" name="piper">
-    <xacro:arg name="initial_positions_file" default="initial_positions.yaml" />
-    <!-- Import piper urdf file -->
-    <xacro:include filename="$(find piper_description)/urdf/piper_description.xacro" />
-    <!-- Import control_xacro -->
-    <xacro:include filename="piper.ros2_control.xacro" />
-    <xacro:piper_ros2_control name="FakeSystem" initial_positions_file="$(arg initial_positions_file)"/>
+  <!-- Arguments -->
+  <xacro:arg name="initial_positions_file" default="initial_positions.yaml" />
+  <xacro:arg name="fake_hardware" default="true"/>
+  <!-- Vollständiges URDF mit Gripper -->
+  <xacro:include filename="$(find piper_description)/urdf/piper_description.xacro" />
+  <!-- ros2_control-Xacro einbinden -->
+  <xacro:include filename="piper.ros2_control.xacro" />
+  <!-- ros2_control-Makro aufrufen -->
+  <xacro:piper_ros2_control
+      name="piper_hw"
+      initial_positions_file="$(arg initial_positions_file)"
+      fake_hardware="$(arg fake_hardware)" />
 </robot>

Commit message: changed gripper config. gripper controller is missing. need to be implemented.

File: ros2_ws/src/piper_ros/src/piper_description/urdf/piper_description.urdf (robot description, URDF)
Before this commit: robot piper, 10 links, 9 joints
Joints:
- joint joint8: mimic joint=joint7 multiplier=-1 offset=0 -> (none)
