Commit message: ros2 fake controller allows gripper actions for simulation

File: ros2_ws/src/piper_ros/src/piper_description/urdf/piper_description.xacro (robot description, xacro)
@@ -503,4 +503,5 @@
       effort="10"
       velocity="1" />
+    <mimic joint="joint7" multiplier="-1.0" offset="0.0"/>
   </joint>
 <!-- controller -->

Commit message: robot movement and gripper movement are now working perfectly

File: ros2_ws/src/piper_ros/src/piper_description/urdf/piper_description.xacro (robot description, xacro)
@@ -489,19 +489,10 @@
     name="joint8"
     type="prismatic">
-    <origin
-      xyz="0 0 0.1358"
-      rpy="1.5708 0 -3.1416" />
-    <parent
-      link="gripper_base" />
-    <child
-      link="link8" />
-    <axis
-      xyz="0 0 -1" />
-    <limit
-      lower="-0.035"
-      upper="0"
-      effort="10"
-      velocity="1" />
-    <mimic joint="joint7" multiplier="-1.0" offset="0.0"/>
+    <origin xyz="0 0 0.1358" rpy="1.5708 0 -3.1416" />
+    <parent link="gripper_base" />
+    <child link="link8" />
+    <axis xyz="0 0 -1" />
+    <limit lower="-0.035" upper="0.0" effort="10" velocity="1" />
+    <!-- <mimic joint="joint7" multiplier="-1.0" offset="0.0"/> -->
   </joint>
 <!-- controller -->

File: ros2_ws/src/piper_ros/src/piper_moveit/piper_with_gripper_moveit/config/piper.ros2_control.xacro (robot description, xacro)
@@ -64,4 +64,11 @@
         <state_interface name="velocity"/>
       </joint>
+      <joint name="joint8">
+        <command_interface name="position"/>
+        <state_interface name="position">
+          <param name="initial_value">${initial_positions['joint8']}</param>
+        </state_interface>
+        <state_interface name="velocity"/>
+      </joint>
     </ros2_control>
   </xacro:macro>

Commit message: created scene for pick and place application. first test with moveit2 and issac sim to pick can and replaced it.

File: ros2_ws/src/piper_ros/src/piper_description/urdf/piper_description.xacro (robot description, xacro)
@@ -7,5 +7,12 @@
   <joint name="fixed_base_joint" type="fixed">
       <parent link="world"/>
+      <child link="base_offset"/>
+  </joint>
+<!-- base offset (nvidia issac sim) -->
+  <link name="base_offset"/>
+  <joint name="fixed_base_joint2" type="fixed">
+      <parent link="base_offset"/>
       <child link="base_link"/>
+      <origin xyz="0.34592 0.0 0.76" rpy="0 0 0"/>
   </joint>
 <!-- arm -->
@@ -387,4 +394,11 @@
     <child
       link="gripper_base" />
+  </joint>
+  <!-- endeffector offset -->
+  <link name="ee_offset"/>
+  <joint name="ee_joint" type="fixed">
+      <parent link="gripper_base"/>
+      <child link="ee_offset"/>
+      <origin xyz="0.0 0.0 0.08" rpy="0 0 0"/>
   </joint>
   <link

Commit message: implementation of greb and rotate the wheel rim. need to be tested with isaac sim environment.

File: ros2_ws/src/piper_ros/src/piper_description/urdf/piper_description.xacro (robot description, xacro)
@@ -14,5 +14,5 @@
       <parent link="base_offset"/>
       <child link="base_link"/>
-      <origin xyz="0.34592 0.0 0.76" rpy="0 0 0"/>
+      <origin xyz="0.19097 0.0 0.76" rpy="0 0 0"/>
   </joint>
 <!-- arm -->

Commit message: Adjusted the configuration. Robot movement still in progress.

File: ros2_ws/src/piper_ros/src/piper_description/urdf/piper_description.xacro (robot description, xacro)
@@ -16,4 +16,5 @@
       <origin xyz="0.19097 0.0 0.76" rpy="0 0 0"/>
   </joint>
+<!-- <origin xyz="0.34592 0.0 0.76" rpy="0 0 0"/> -->
 <!-- arm -->
 <link

Commit message: improved the grab and rotate movement

File: ros2_ws/src/piper_ros/src/piper_description/urdf/piper_description.xacro (robot description, xacro)
@@ -14,6 +14,7 @@
       <parent link="base_offset"/>
       <child link="base_link"/>
-      <origin xyz="0.19097 0.0 0.76" rpy="0 0 0"/>
-  </joint>
+      <origin xyz="0.10397 0.0 0.76" rpy="0 0 0"/>
+  </joint>
+<!-- <origin xyz="0.19097 0.0 0.76" rpy="0 0 0"/> -->
 <!-- <origin xyz="0.34592 0.0 0.76" rpy="0 0 0"/> -->
 <!-- arm -->

Commit message: changed paramters. added material for friction. optimized position. tested simulation.

File: ros2_ws/src/piper_ros/src/piper_description/urdf/piper_description.xacro (robot description, xacro)
@@ -398,9 +398,9 @@
   </joint>
   <!-- endeffector offset -->
-  <link name="ee_offset"/>
+  <link name="ee_tcp"/>
   <joint name="ee_joint" type="fixed">
       <parent link="gripper_base"/>
-      <child link="ee_offset"/>
-      <origin xyz="0.0 0.0 0.08" rpy="0 0 0"/>
+      <child link="ee_tcp"/>
+      <origin xyz="0.0 0.0 0.10" rpy="0 0 0"/>
   </joint>
   <link
@@ -459,5 +459,5 @@
       lower="0"
       upper="0.035"
-      effort="10"
+      effort="50"
       velocity="1" />
   </joint>
@@ -509,5 +509,5 @@
     <child link="link8" />
     <axis xyz="0 0 -1" />
-    <limit lower="-0.035" upper="0.0" effort="10" velocity="1" />
+    <limit lower="-0.035" upper="0.0" effort="50" velocity="1" />
     <!-- <mimic joint="joint7" multiplier="-1.0" offset="0.0"/> -->
   </joint>

Commit message: update main form remote pc

File: ros2_ws/src/piper_ros/src/piper_description/urdf/piper_description.xacro (robot description, xacro)
@@ -16,6 +16,4 @@
       <origin xyz="0.10397 0.0 0.76" rpy="0 0 0"/>
   </joint>
-<!-- <origin xyz="0.19097 0.0 0.76" rpy="0 0 0"/> -->
-<!-- <origin xyz="0.34592 0.0 0.76" rpy="0 0 0"/> -->
 <!-- arm -->
 <link
